Commit message: Updated Tutorial for using sensors with Holonomic Configuration

File: Tutorials/SoftwareInstallation/RobotX Simulation/vmrc_ws/build/vmrc/wamv_gazebo/urdf/wamv_gazebo_sensors.urdf (robot description, URDF)
Before this commit: robot WAM-V, 10 links, 9 joints
Links:
- removed link left_engine_link
- removed link left_propeller_link
- removed link right_engine_link
- removed link right_propeller_link
- added link left_front_engine_link, mass 15; collision box size=0.12 0.15 0.12; collision box size=0.2 0.15 0.83
- added link left_front_propeller_link, mass 0.5; collision cylinder length=0.18 radius=0.24; visual mesh filename=package://wamv_description/mesh/propeller.dae
- added link left_rear_engine_link, mass 15; collision box size=0.12 0.15 0.12; collision box size=0.2 0.15 0.83
- added link left_rear_propeller_link, mass 0.5; collision cylinder length=0.18 radius=0.24; visual mesh filename=package://wamv_description/mesh/propeller.dae
- added link right_front_engine_link, mass 15; collision box size=0.12 0.15 0.12; collision box size=0.2 0.15 0.83
- added link right_front_propeller_link, mass 0.5; collision cylinder length=0.18 radius=0.24; visual mesh filename=package://wamv_description/mesh/propeller.dae
- added link right_rear_engine_link, mass 15; collision box size=0.12 0.15 0.12; collision box size=0.2 0.15 0.83
- added link right_rear_propeller_link, mass 0.5; collision cylinder length=0.18 radius=0.24; visual mesh filename=package://wamv_description/mesh/propeller.dae
Joints:
- removed joint left_chasis_engine_joint
- removed joint left_engine_propeller_joint
- removed joint right_chasis_engine_joint
- removed joint right_engine_propeller_joint
- added joint left_front_chasis_engine_joint: type fixed, parent base_link, child left_front_engine_link, origin xyz=1.6 0.7  0.25 rpy=0.0 0.0 -0.785
- added joint left_front_engine_propeller_joint: type continuous, parent left_front_engine_link, child left_front_propeller_link, origin xyz=-0.278156 0 -0.509371 rpy=0 0 0, axis 1 0 0, limit effort=100 velocity=100
- added joint left_rear_chasis_engine_joint: type fixed, parent base_link, child left_rear_engine_link, origin xyz=-2.373776 1.027135 0.318237 rpy=0.0 0.0 0.785
- added joint left_rear_engine_propeller_joint: type continuous, parent left_rear_engine_link, child left_rear_propeller_link, origin xyz=-0.278156 0 -0.509371 rpy=0 0 0, axis 1 0 0, limit effort=100 velocity=100
- added joint right_front_chasis_engine_joint: type fixed, parent base_link, child right_front_engine_link, origin xyz=1.6 -0.7 0.25 rpy=0.0 0.0 +0.785
- added joint right_front_engine_propeller_joint: type continuous, parent right_front_engine_link, child right_front_propeller_link, origin xyz=-0.278156 0 -0.509371 rpy=0 0 0, axis 1 0 0, limit effort=100 velocity=100
- added joint right_rear_chasis_engine_joint: type fixed, parent base_link, child right_rear_engine_link, origin xyz=-2.373776 -1.027135 0.318237 rpy=0.0 0.0 -0.785
- added joint right_rear_engine_propeller_joint: type continuous, parent right_rear_engine_link, child right_rear_propeller_link, origin xyz=-0.278156 0 -0.509371 rpy=0 0 0, axis 1 0 0, limit effort=100 velocity=100

File: Tutorials/SoftwareInstallation/RobotX Simulation/vmrc_ws/devel/share/wamv_gazebo/urdf/wamv_gazebo.urdf (robot description, URDF)
Before this commit: robot WAM-V, 5 links, 4 joints
Links:
- removed link left_engine_link
- removed link left_propeller_link
- removed link right_engine_link
- removed link right_propeller_link
- added link left_front_engine_link, mass 15; collision box size=0.12 0.15 0.12; collision box size=0.2 0.15 0.83
- added link left_front_propeller_link, mass 0.5; collision cylinder length=0.18 radius=0.24; visual mesh filename=package://wamv_description/mesh/propeller.dae
- added link left_rear_engine_link, mass 15; collision box size=0.12 0.15 0.12; collision box size=0.2 0.15 0.83
- added link left_rear_propeller_link, mass 0.5; collision cylinder length=0.18 radius=0.24; visual mesh filename=package://wamv_description/mesh/propeller.dae
- added link right_front_engine_link, mass 15; collision box size=0.12 0.15 0.12; collision box size=0.2 0.15 0.83
- added link right_front_propeller_link, mass 0.5; collision cylinder length=0.18 radius=0.24; visual mesh filename=package://wamv_description/mesh/propeller.dae
- added link right_rear_engine_link, mass 15; collision box size=0.12 0.15 0.12; collision box size=0.2 0.15 0.83
- added link right_rear_propeller_link, mass 0.5; collision cylinder length=0.18 radius=0.24; visual mesh filename=package://wamv_description/mesh/propeller.dae
Joints:
- removed joint left_chasis_engine_joint
- removed joint left_engine_propeller_joint
- removed joint right_chasis_engine_joint
- removed joint right_engine_propeller_joint
- added joint left_front_chasis_engine_joint: type fixed, parent base_link, child left_front_engine_link, origin xyz=1.6 0.7  0.25 rpy=0.0 0.0 -0.785
- added joint left_front_engine_propeller_joint: type continuous, parent left_front_engine_link, child left_front_propeller_link, origin xyz=-0.278156 0 -0.509371 rpy=0 0 0, axis 1 0 0, limit effort=100 velocity=100
- added joint left_rear_chasis_engine_joint: type fixed, parent base_link, child left_rear_engine_link, origin xyz=-2.373776 1.027135 0.318237 rpy=0.0 0.0 0.785
- added joint left_rear_engine_propeller_joint: type continuous, parent left_rear_engine_link, child left_rear_propeller_link, origin xyz=-0.278156 0 -0.509371 rpy=0 0 0, axis 1 0 0, limit effort=100 velocity=100
- added joint right_front_chasis_engine_joint: type fixed, parent base_link, child right_front_engine_link, origin xyz=1.6 -0.7 0.25 rpy=0.0 0.0 +0.785
- added joint right_front_engine_propeller_joint: type continuous, parent right_front_engine_link, child right_front_propeller_link, origin xyz=-0.278156 0 -0.509371 rpy=0 0 0, axis 1 0 0, limit effort=100 velocity=100
- added joint right_rear_chasis_engine_joint: type fixed, parent base_link, child right_rear_engine_link, origin xyz=-2.373776 -1.027135 0.318237 rpy=0.0 0.0 -0.785
- added joint right_rear_engine_propeller_joint: type continuous, parent right_rear_engine_link, child right_rear_propeller_link, origin xyz=-0.278156 0 -0.509371 rpy=0 0 0, axis 1 0 0, limit effort=100 velocity=100

File: Tutorials/SoftwareInstallation/RobotX Simulation/vmrc_ws/src/vmrc/wamv_gazebo/urdf/my_wamv.urdf (robot description, URDF)
Before this commit: robot WAM-V, 13 links, 12 joints
Links:
- removed link left_engine_link
- removed link left_propeller_link
- removed link right_engine_link
- removed link right_propeller_link
- added link left_front_engine_link, mass 15; collision box size=0.12 0.15 0.12; collision box size=0.2 0.15 0.83
- added link left_front_propeller_link, mass 0.5; collision cylinder length=0.18 radius=0.24; visual mesh filename=package://wamv_description/mesh/propeller.dae
- added link left_rear_engine_link, mass 15; collision box size=0.12 0.15 0.12; collision box size=0.2 0.15 0.83
- added link left_rear_propeller_link, mass 0.5; collision cylinder length=0.18 radius=0.24; visual mesh filename=package://wamv_description/mesh/propeller.dae
- added link lidar_wamv_link; visual cylinder length=0.1 radius=0.025
- added link right_front_engine_link, mass 15; collision box size=0.12 0.15 0.12; collision box size=0.2 0.15 0.83
- added link right_front_propeller_link, mass 0.5; collision cylinder length=0.18 radius=0.24; visual mesh filename=package://wamv_description/mesh/propeller.dae
- added link right_rear_engine_link, mass 15; collision box size=0.12 0.15 0.12; collision box size=0.2 0.15 0.83
- added link right_rear_propeller_link, mass 0.5; collision cylinder length=0.18 radius=0.24; visual mesh filename=package://wamv_description/mesh/propeller.dae
Joints:
- removed joint left_chasis_engine_joint
- removed joint left_engine_propeller_joint
- removed joint right_chasis_engine_joint
- removed joint right_engine_propeller_joint
- added joint left_front_chasis_engine_joint: type fixed, parent base_link, child left_front_engine_link, origin xyz=1.6 0.7  0.25 rpy=0.0 0.0 -0.785
- added joint left_front_engine_propeller_joint: type continuous, parent left_front_engine_link, child left_front_propeller_link, origin xyz=-0.278156 0 -0.509371 rpy=0 0 0, axis 1 0 0, limit effort=100 velocity=100
- added joint left_rear_chasis_engine_joint: type fixed, parent base_link, child left_rear_engine_link, origin xyz=-2.373776 1.027135 0.318237 rpy=0.0 0.0 0.785
- added joint left_rear_engine_propeller_joint: type continuous, parent left_rear_engine_link, child left_rear_propeller_link, origin xyz=-0.278156 0 -0.509371 rpy=0 0 0, axis 1 0 0, limit effort=100 velocity=100
- added joint lidar_wamv_joint: type fixed, parent base_link, child lidar_wamv_link, origin xyz=0.5 -0.3 2 rpy=0 0 0
- added joint right_front_chasis_engine_joint: type fixed, parent base_link, child right_front_engine_link, origin xyz=1.6 -0.7 0.25 rpy=0.0 0.0 +0.785
- added joint right_front_engine_propeller_joint: type continuous, parent right_front_engine_link, child right_front_propeller_link, origin xyz=-0.278156 0 -0.509371 rpy=0 0 0, axis 1 0 0, limit effort=100 velocity=100
- added joint right_rear_chasis_engine_joint: type fixed, parent base_link, child right_rear_engine_link, origin xyz=-2.373776 -1.027135 0.318237 rpy=0.0 0.0 -0.785
- added joint right_rear_engine_propeller_joint: type continuous, parent right_rear_engine_link, child right_rear_propeller_link, origin xyz=-0.278156 0 -0.509371 rpy=0 0 0, axis 1 0 0, limit effort=100 velocity=100
- joint front_camera_joint: origin xyz=0.5 0 1.5 rpy=0 0 0 -> xyz=0.75 0.3 1.5 rpy=0 0.261799387799 0
- joint gps_wamv_joint: origin xyz=0 0 1.3 rpy=0 0 0 -> xyz=0 0.2 1.3 rpy=0 0 0
- joint imu_wamv_joint: origin xyz=0 0 1.3 rpy=0 0 0 -> xyz=0 -0.2 1.3 rpy=0 0 0

File: Tutorials/SoftwareInstallation/RobotX Simulation/vmrc_ws/src/vmrc/wamv_gazebo/urdf/my_wamv.urdf.xacro (robot description, xacro)
@@ -2,15 +2,32 @@
 <robot xmlns:xacro="http://ros.org/wiki/xacro"
        name="WAM-V">
+  <xacro:arg name="camera_enabled" default="true" />
+  <xacro:arg name="gps_enabled" default="true" />
+  <xacro:arg name="imu_enabled" default="true" />
+  <xacro:arg name="lidar_enabled" default="true" />
+  <xacro:arg name="ground_truth_enabled" default="true" />
   <!-- Basic frame of WAM-V -->
   <xacro:include filename="$(find wamv_gazebo)/urdf/wamv_gazebo.urdf.xacro" />
   <!-- ADD SENSORS -->
   <!-- Add a front camera -->
-  <xacro:wamv_camera name="front_camera"/>
+  <xacro:if value="$(arg camera_enabled)">
+    <xacro:wamv_camera name="front_camera" y="0.3" x="0.75" P="${radians(15)}" />
+  </xacro:if>
   <!-- Add simulated GPS -->
-  <xacro:wamv_gps name="gps_wamv"/>
+  <xacro:if value="$(arg gps_enabled)">
+    <xacro:wamv_gps name="gps_wamv" y="0.2" />
+  </xacro:if>
   <!-- Add Simulated IMU -->
-  <xacro:wamv_imu name="imu_wamv"/>
+  <xacro:if value="$(arg imu_enabled)">
+    <xacro:wamv_imu name="imu_wamv" y="-0.2" />
+  </xacro:if>
+  <!-- Add 3D LIDAR -->
+  <xacro:if value="$(arg lidar_enabled)">
+    <xacro:wamv_3d_lidar name="lidar_wamv" y="-0.3" />
+  </xacro:if>
   <!-- Add P3D ground truth -->
-  <xacro:wamv_p3d name="p3d_wamv"/>
+  <xacro:if value="$(arg ground_truth_enabled)">
+    <xacro:wamv_p3d name="p3d_wamv"/>
+  </xacro:if>
   <xacro:property name="stereo_x" value="1.0" />
   <xacro:wamv_camera name="stereo_left" x="${stereo_x}" y="0.3" z="1.5" P="${radians(15)}" />

File: Tutorials/SoftwareInstallation/RobotX Simulation/vmrc_ws/src/vmrc/wamv_gazebo/urdf/wamv_gazebo.urdf.xacro (robot description, xacro)
@@ -5,4 +5,4 @@
   <!-- Default WAM-V with two aft thrusters -->
   <xacro:include filename="$(find wamv_gazebo)/urdf/wamv_gazebo.xacro" />
-  <xacro:wamv_gazebo thruster_layout="$(find wamv_gazebo)/urdf/thruster_layouts/wamv_aft_thrusters.xacro"/>
+  <xacro:wamv_gazebo thruster_layout="$(find wamv_gazebo)/urdf/thruster_layouts/wamv_x_thrusters.xacro"/>
 </robot>
